File: dmf.brd (EAGLE design)
At the start: 100 x 100 mm, 64 parts, among them IC1 7805TV, IC3 4504D, IC4 FT232RL, J1 5.5x2.1mm Barrel, J2 FTS-105-01-L-DV, Q1 BUZ11BV, U1 MCP1416T-E/OT, U2 MCP601T-I/OT, U3 ARDUINO_SHIELDNOHOLES, U4 MCP3204-CI/SL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

Commit message: dmf.brd routing
Parts:
- removed L1: (no value), dubres:WE-PD_1260/1245/1280/1210
- added C13: 10uF, rcl:C0805
- added JPI2C1, JPI2C2: (no value), pinhead-2:1X04-S
- added L2: 6.8UH, Panasonic-ELL:IND_ELL5PR
- moved HVOUT 79.7 mm to (67.9, 91.1), turned to 270 degrees
- moved U2 72.5 mm to (72.2, 84.2), turned to 270 degrees
- moved RCSG 68.2 mm to (69.2, 80.2), turned to 270 degrees
- moved RSHUNT 66.8 mm to (68.3, 84.8), turned to 90 degrees
- moved CMCPBP 65.5 mm to (75.3, 84.7), turned to 90 degrees
- moved D3 62.0 mm to (63.7, 81.5), turned to 270 degrees
- moved CVIN 61.3 mm to (7.95, 86.4), turned to 270 degrees
- moved RCSF 61.2 mm to (72.1, 80.6), turned to 180 degrees
- moved C3 53.7 mm to (79.2, 82.3)
- moved LED6 52.6 mm to (60.2, 34.1), turned to 0 degrees
- moved RB5 49.7 mm to (60.2, 37.5), turned to 90 degrees
- moved U4 43.8 mm to (82.0, 77.2), turned to 90 degrees
- moved C1 34.7 mm to (15.1, 83.7)
- moved C2 34.7 mm to (24.2, 81.6)
- moved C4 34.7 mm to (15.8, 90.2)
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Connections:
- removed net A1: U3.A1, U6.33
- new net ADCEX: JPI2C1.4, U4.4
- new net ADCEX2: JPI2C2.4, U3.A1, U6.33
- new net CSENS2: JPI2C2.1, U3.A0, U6.32
- new net VIN_SENS2: JPI2C2.2, U3.A4, U6.40
- new net VOUT_SENS2: JPI2C2.3, U3.A5, U6.42
- net +5V: no longer CMCPBP.1
- net CSENS: now also JPI2C1.1; no longer U3.A0, U6.32
- net GND: now also C13.2
- net N$9: now also L2.1; no longer L1.1
- net V+: now also C13.1, L2.2; no longer L1.2
- net VCC: now also CMCPBP.1
- net VIN_SENS: now also JPI2C1.2; no longer U3.A4, U6.40
- net VOUT_SENS: now also JPI2C1.3; no longer U3.A5, U6.42
Routing:
- net GND: track 196.3 -> 589.8 mm, vias 5 -> 17
- net V+: track 49.4 -> 217.9 mm, vias 2 -> 4
- net VCC: track 102.0 -> 261.1 mm, vias 1 -> 6
- net OUT_CLK: track 40.9 -> 153.3 mm, vias 3 -> 5
- net 3V3: track 15.8 -> 95.3 mm, vias 0 -> 1
- net PWMINPUT: track 24.1 -> 99.9 mm, vias 1 -> 3
- net CSENS2: track 0.00 -> 75.0 mm
- net ADCEX2: track 0.00 -> 71.0 mm, vias 0 -> 1
- net +5V: track 34.8 -> 104.7 mm, vias 0 -> 2
- net VOUT_SENS2: track 0.00 -> 68.5 mm, vias 0 -> 1
- net VIN_SENS2: track 0.00 -> 67.4 mm, vias 0 -> 1
- net HV+: track 0.00 -> 66.1 mm, vias 0 -> 1
- net OUT_DATA: track 71.7 -> 135.4 mm, vias 2 -> 4
- net OUT_POL: track 28.7 -> 72.4 mm, vias 1 -> 2
- net A1: track 32.8 -> 0.00 mm
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- added copper zone on layer 1, net GND
- added copper zone on layer 16, net GND

Commit message: * DMF board first iteration
Parts:
- added HVIN: (no value), pinhead-2:1X02
- CVIN, CVOUT: device rcl:E5-8,5 -> rcl:E7,5-18
- L2: value 6.8UH -> 1.0UH; device Panasonic-ELL:IND_ELL5PR -> Panasonic-ELL:IND_ELL6XH
- U4: value MCP3204-CI/SL -> MCP3204
- moved RCSG1 27.3 mm to (84.4, 86.9), turned to 90 degrees
- moved D2 16.2 mm to (76.6, 89.6), turned to 0 degrees
- moved CVIN 14.9 mm to (10.9, 71.8), turned to 0 degrees
- moved CVOUT 4.60 mm to (55.8, 90.6)
- moved HVOUT 4.39 mm to (68.3, 95.5)
- moved D3 2.88 mm to (64.0, 78.7)
Connections:
- net N$16 renamed SCL
- net N$22 renamed SDA
- net GND: now also HVIN.2
- net HV+: now also HVIN.1
Routing:
- net HV+: track 66.1 -> 88.4 mm
- net HVGND: track 12.6 -> 21.0 mm
- net GND: track 589.8 -> 596.3 mm, vias 17 -> 18
- net N$7: track 0.00 -> 2.96 mm
- net N$41: track 7.72 -> 10.1 mm
Other:
- board text added: "+"
- board text added: "3v3"
- board text added: "5V"
- board text added: "5v"
- board text added: "GND"
- board text added: "ICSKIP"
- board text added: "ISPT"
- board text added: "RX"
- board text added: "RXD"
- board text added: "SCL"
- board text added: "SDA"
- board text added: "TX"
- board text added: "TXD"
- board text added: "VCC"
- board text added: "VSEL"
- board text added: "adcex"
- board text added: "clk"
- board text added: "cs"
- board text added: "data"
- board text added: "gnd"
- board text added: "latch"
- board text added: "pol"
- board text added: "vcc"
- board text added: "vins"
- board text added: "vouts"
