File: dmf.sch (EAGLE design)
At the start: 64 parts, among them IC1 7805TV, IC3 4504D, IC4 FT232RL, J1 5.5x2.1mm Barrel, J2 FTS-105-01-L-DV, Q1 BUZ11BV, U1 MCP1416T-E/OT, U2 MCP601T-I/OT, U3 ARDUINO_SHIELDNOHOLES, U4 MCP3204-CI/SL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

Commit message: dmf.brd routing
Parts:
- removed L1: (no value), dubres:WE-PD-74477001_1260/1245/1280/1210
- added C13: 10uF, rcl:C-EUC0805
- added JPI2C1, JPI2C2: (no value), pinhead-2:PINHD-1X04_2.54-S
- added L2: 6.8UH, Panasonic-ELL:ELL5PR6R8N-5PR
Connections:
- removed net A1: U3.A1, U6.TMS/PIO0_12/AD1/CT32B1_CAP0
- new net ADCEX: JPI2C1.4, U4.CH3
- new net ADCEX2: JPI2C2.4, U3.A1, U6.TMS/PIO0_12/AD1/CT32B1_CAP0
- new net CSENS2: JPI2C2.1, U3.A0, U6.TDI/PIO0_11/AD0/CT32B0_MAT3
- new net VIN_SENS2: JPI2C2.2, U3.A4, U6.PIO0_16/AD5/CT32B1_MAT3/WAKEUP
- new net VOUT_SENS2: JPI2C2.3, U3.A5, U6.PIO0_23/AD7
- net +5V: no longer CMCPBP.1
- net CSENS: now also JPI2C1.1; no longer U3.A0, U6.TDI/PIO0_11/AD0/CT32B0_MAT3
- net GND: now also C13.2
- net N$9: now also L2.1; no longer L1.1
- net V+: now also C13.1, L2.2; no longer L1.2
- net VCC: now also CMCPBP.1
- net VIN_SENS: now also JPI2C1.2; no longer U3.A4, U6.PIO0_16/AD5/CT32B1_MAT3/WAKEUP
- net VOUT_SENS: now also JPI2C1.3; no longer U3.A5, U6.PIO0_23/AD7

Commit message: * DMF board first iteration
Parts:
- added HVIN: (no value), pinhead-2:PINHD-1X02_2.54
- CVIN, CVOUT: device rcl:CPOL-EUE5-8.5 -> rcl:CPOL-EUE7.5-18
- L2: value 6.8UH -> 1.0UH; device Panasonic-ELL:ELL5PR6R8N-5PR -> Panasonic-ELL:ELL6RH1R0M-6XH
- U4: value MCP3204-CI/SL -> MCP3204
Connections:
- net N$16 renamed SCL
- net N$22 renamed SDA
- net GND: now also HVIN.2
- net HV+: now also HVIN.1
Changed lines of the file:
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@@
 <part name="C2" library="rcl" deviceset="C-EU" device="C0805" value="1nF"/>
 <part name="R6" library="rcl" deviceset="R-EU_" device="R0603" value="50k"/>
-<part name="CVOUT" library="rcl" deviceset="CPOL-EU" device="E5-8.5"/>
+<part name="CVOUT" library="rcl" deviceset="CPOL-EU" device="E7.5-18"/>
 <part name="C4" library="rcl" deviceset="C-EU" device="C0805"/>
 <part name="R7" library="rcl" deviceset="R-EU_" device="R0603"/>
@@
 <part name="P+9" library="supply1" deviceset="VCC" device=""/>
 <part name="J2" library="hvgen" deviceset="FTS-105-01-L-DV" device=""/>
-<part name="CVIN" library="rcl" deviceset="CPOL-EU" device="E5-8.5"/>
+<part name="CVIN" library="rcl" deviceset="CPOL-EU" device="E7.5-18"/>
 <part name="C6" library="rcl" deviceset="C-EU" device="C1206" value="47uF"/>
 <part name="C14" library="rcl" deviceset="C-EU" device="C0805" value="100n"/>
@@
 <part name="IC1" library="linear" deviceset="78*" device="TV" technology="05"/>
 <part name="D3" library="diode" deviceset="ZENER-DIODE" device="SMB" value="3v3"/>
-<part name="U4" library="hvgen" deviceset="MCP3204-CI/SL" device=""/>
+<part name="U4" library="hvgen" deviceset="MCP3204-CI/SL" device="" value="MCP3204"/>
 <part name="GND14" library="supply1" deviceset="GND" device=""/>
 <part name="P+4" library="supply1" deviceset="VCC" device=""/>
 <part name="C3" library="rcl" deviceset="C-EU" device="C0805" value="1uF"/>
-<part name="L2" library="Panasonic-ELL" deviceset="ELL" device="-5PR" technology="5PR6R8N" value=" 6.8UH "/>
+<part name="L2" library="Panasonic-ELL" deviceset="ELL" device="-6XH" technology="6RH1R0M" value="1.0UH"/>
 <part name="C13" library="rcl" deviceset="C-EU" device="C0805" value="10uF"/>
 <part name="P+12" library="supply1" deviceset="VCC" device=""/>
 <part name="JPI2C1" library="pinhead-2" deviceset="PINHD-1X04" device="_2.54-S"/>
 <part name="JPI2C2" library="pinhead-2" deviceset="PINHD-1X04" device="_2.54-S"/>
+<part name="HVIN" library="pinhead-2" deviceset="PINHD-1X02" device="_2.54"/>
 </parts>
 <sheets>
@@
 <instance part="JPI2C1" gate="A" x="106.68" y="144.78"/>
 <instance part="JPI2C2" gate="A" x="96.52" y="144.78"/>
+<instance part="HVIN" gate="A" x="5.08" y="53.34"/>
 </instances>
 <busses>
@@
 <junction x="-96.52" y="40.64"/>
 <pinref part="U1" gate="A" pin="GND"/>
-<wire x1="10.16" y1="5.08" x2="-12.7" y2="5.08" width="0.1524" layer="91"/>
+<wire x1="10.16" y1="5.08" x2="2.54" y2="5.08" width="0.1524" layer="91"/>
+<wire x1="2.54" y1="5.08" x2="-12.7" y2="5.08" width="0.1524" layer="91"/>
 <wire x1="-78.74" y1="43.18" x2="-91.44" y2="43.18" width="0.1524" layer="91"/>
 <wire x1="-91.44" y1="43.18" x2="-91.44" y2="40.64" width="0.1524" layer="91"/>
@@
 <pinref part="C13" gate="G$1" pin="2"/>
 <wire x1="-78.74" y1="17.78" x2="-78.74" y2="5.08" width="0.1524" layer="91"/>
+<pinref part="HVIN" gate="A" pin="2"/>
+<wire x1="2.54" y1="53.34" x2="2.54" y2="5.08" width="0.1524" layer="91"/>
 </segment>
 <segment>
@@
 <label x="33.02" y="71.12" size="1.778" layer="95"/>
 <pinref part="D2" gate="1" pin="C"/>
-<wire x1="10.16" y1="71.12" x2="-12.7" y2="71.12" width="0.1524" layer="91"/>
+<wire x1="10.16" y1="71.12" x2="2.54" y2="71.12" width="0.1524" layer="91"/>
+<wire x1="2.54" y1="71.12" x2="-12.7" y2="71.12" width="0.1524" layer="91"/>
 <wire x1="10.16" y1="43.18" x2="10.16" y2="71.12" width="0.1524" layer="91"/>
 <pinref part="RBLEED" gate="G$1" pin="2"/>
 <wire x1="-12.7" y1="55.88" x2="-5.08" y2="55.88" width="0.1524" layer="91"/>
 <wire x1="-5.08" y1="55.88" x2="-5.08" y2="48.26" width="0.1524" layer="91"/>
+<pinref part="HVIN" gate="A" pin="1"/>
+<wire x1="2.54" y1="55.88" x2="2.54" y2="71.12" width="0.1524" layer="91"/>
 </segment>
 </net>
@@
 </segment>
 </net>
-<net name="N$16" class="0">
+<net name="SCL" class="0">
 <segment>
 <pinref part="JPI2C" gate="A" pin="3"/>
@@
 </segment>
 </net>
-<net name="N$22" class="0">
+<net name="SDA" class="0">
 <segment>
 <pinref part="U6" gate="A" pin="PIO0_5/SDA"/>
@@
 </nets>
 </sheet>
+<sheet>
+<plain>
+</plain>
+<instances>
+</instances>
+<busses>
+</busses>
+<nets>
+</nets>
+</sheet>
