File: hv507_connector.brd (EAGLE design)
At the start: 50 x 50 mm, 10 parts

Commit message: * DMF board first iteration
Connections:
- net N$1 renamed 16
- net N$16 renamed 1
- net N$17 renamed 32
- net N$32 renamed 17
- net N$33 renamed 64
- net N$48 renamed 49
- net N$49 renamed 40
- net N$56 renamed 33
- net N$57 renamed 48
- net N$64 renamed 41
Other:
- board size 50 x 50 mm -> 90 x 50 mm
- board text added: "47"
- board text added: "63"
- board text added: "CLK"
- board text added: "DATA"
- board text added: "GND"
- board text added: "HV507 connector"
- board text added: "High Voltage"
- board text added: "LATCH"
- board text added: "POL"
- board text added: "VDD"
- board text added: "VPP"
Changed lines of the file:
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@@
 <layer number="44" name="Drills" color="7" fill="1" visible="no" active="yes"/>
 <layer number="45" name="Holes" color="7" fill="1" visible="yes" active="yes"/>
-<layer number="46" name="Milling" color="3" fill="1" visible="no" active="yes"/>
+<layer number="46" name="Milling" color="3" fill="1" visible="yes" active="yes"/>
 <layer number="47" name="Measures" color="7" fill="1" visible="no" active="yes"/>
 <layer number="48" name="Document" color="7" fill="1" visible="yes" active="yes"/>
@@
 <board>
 <plain>
-<wire x1="0" y1="0" x2="50" y2="0" width="0" layer="20"/>
-<wire x1="50" y1="0" x2="50" y2="50" width="0" layer="20"/>
-<wire x1="50" y1="50" x2="0" y2="50" width="0" layer="20"/>
-<wire x1="0" y1="50" x2="0" y2="0" width="0" layer="20"/>
+<wire x1="-20" y1="0" x2="70" y2="0" width="0" layer="20"/>
+<wire x1="70" y1="0" x2="70" y2="50" width="0" layer="20"/>
+<wire x1="70" y1="50" x2="-20" y2="50" width="0" layer="20"/>
+<wire x1="-20" y1="50" x2="-20" y2="0" width="0" layer="20"/>
 <hole x="3.5" y="10" drill="3"/>
 <hole x="46.5" y="10" drill="3"/>
 <hole x="46.5" y="40" drill="3"/>
 <hole x="3.5" y="40" drill="3"/>
+<text x="46.5" y="15" size="0.8128" layer="21" rot="R180">High
+Voltage</text>
+<text x="48.2" y="16.9" size="0.8128" layer="21" rot="R270">VPP</text>
+<text x="48.2" y="19.8" size="0.8128" layer="21" rot="R270">GND</text>
+<text x="48.5" y="22.5" size="0.8128" layer="21">DATA</text>
+<text x="48.5" y="25" size="0.8128" layer="21">CLK</text>
+<text x="48.5" y="27.5" size="0.8128" layer="21">LATCH</text>
+<text x="48.5" y="30" size="0.8128" layer="21">POL</text>
+<text x="48.5" y="32.5" size="0.8128" layer="21">VDD</text>
+<text x="48.5" y="35" size="0.8128" layer="21">GND</text>
+<text x="45.6" y="3.5" size="0.8128" layer="21">47</text>
+<text x="45.6" y="0.9" size="0.8128" layer="21">63</text>
+<text x="29.2" y="60.6" size="0.8128" layer="21">63</text>
+<text x="29.2" y="60.6" size="0.8128" layer="21">63</text>
+<text x="71.1" y="17.7" size="0.8128" layer="21">63</text>
+<hole x="66.5" y="40" drill="3"/>
+<hole x="66.5" y="10" drill="3"/>
+<hole x="-16.5" y="10" drill="3"/>
+<hole x="-16.5" y="40" drill="3"/>
+<wire x1="56.5" y1="35.5" x2="56.5" y2="22.5" width="6.4516" layer="46"/>
+<text x="-18" y="2" size="1.778" layer="21">HV507 connector</text>
 </plain>
 <attributes>
@@
 </autorouter>
 <elements>
-<element name="JP1" library="pinhead-2" package="1X16-S" value="" x="25" y="45.58"/>
-<element name="JP2" library="pinhead-2" package="1X16-S" value="" x="25" y="48.12"/>
-<element name="JP3" library="pinhead-2" package="1X16-S" value="" x="25" y="1.32" rot="R180"/>
-<element name="JP4" library="pinhead-2" package="1X08-S" value="" x="14.84" y="3.86"/>
-<element name="JP5" library="pinhead-2" package="1X08-S" value="" x="35.16" y="3.86" rot="R180"/>
+<element name="JP1" library="pinhead-2" package="1X16-S" value="" x="25" y="45.58" smashed="yes">
+<attribute name="VALUE" x="4.68" y="42.405" size="1.27" layer="27"/>
+</element>
+<element name="JP2" library="pinhead-2" package="1X16-S" value="" x="25" y="48.12" smashed="yes">
+<attribute name="VALUE" x="4.68" y="44.945" size="1.27" layer="27"/>
+</element>
+<element name="JP3" library="pinhead-2" package="1X16-S" value="" x="25" y="1.32" smashed="yes" rot="R180">
+<attribute name="VALUE" x="45.32" y="4.495" size="1.27" layer="27" rot="R180"/>
+</element>
+<element name="JP4" library="pinhead-2" package="1X08-S" value="" x="14.84" y="3.86" smashed="yes">
+<attribute name="VALUE" x="4.68" y="0.685" size="1.27" layer="27"/>
+</element>
+<element name="JP5" library="pinhead-2" package="1X08-S" value="" x="35.16" y="3.86" smashed="yes" rot="R180">
+<attribute name="VALUE" x="45.32" y="7.035" size="1.27" layer="27" rot="R180"/>
+</element>
 <element name="U$1" library="HV507" package="HV507PG-G" value="HV507" x="25" y="26.72"/>
-<element name="JP6" library="pinhead-2" package="1X06-S" value="" x="46.5" y="29" rot="R90"/>
-<element name="JP7" library="pinhead-2" package="1X02-S" value="" x="46.5" y="17" rot="R90"/>
-<element name="C1" library="rcl" package="C1812" value="" x="40.8" y="18.1" rot="R180"/>
-<element name="C2" library="rcl" package="C1206" value="" x="41.7" y="33.2" rot="R180"/>
+<element name="JP6" library="pinhead-2" package="1X06-S" value="" x="46.5" y="29" smashed="yes" rot="R90">
+<attribute name="VALUE" x="49.675" y="21.38" size="1.27" layer="27" rot="R90"/>
+</element>
+<element name="JP7" library="pinhead-2" package="1X02-S" value="" x="46.5" y="17" smashed="yes" rot="R90">
+<attribute name="VALUE" x="49.675" y="14.46" size="1.27" layer="27" rot="R90"/>
+</element>
+<element name="C1" library="rcl" package="C1812" value="" x="40.8" y="18.1" smashed="yes" rot="R180">
+<attribute name="NAME" x="40.405" y="15.86" size="1.27" layer="25" rot="R180"/>
+<attribute name="VALUE" x="42.705" y="21.91" size="1.27" layer="27" rot="R180"/>
+</element>
+<element name="C2" library="rcl" package="C1206" value="" x="41.7" y="33.2" smashed="yes" rot="R180">
+<attribute name="NAME" x="41.67" y="35.63" size="1.27" layer="25" rot="R180"/>
+<attribute name="VALUE" x="42.97" y="35.74" size="1.27" layer="27" rot="R180"/>
+</element>
 </elements>
 <signals>
-<signal name="N$1">
+<signal name="16">
 <contactref element="U$1" pad="56"/>
 <contactref element="JP1" pad="1"/>
@@
 <wire x1="41.86" y1="45.23" x2="41.51" y2="45.58" width="0.3048" layer="1"/>
 </signal>
-<signal name="N$16">
+<signal name="1">
 <contactref element="U$1" pad="41"/>
 <contactref element="JP1" pad="16"/>
@@
 <wire x1="43.28" y1="44.81" x2="44.05" y2="45.58" width="0.3048" layer="1"/>
 </signal>
-<signal name="N$17">
+<signal name="32">
 <contactref element="U$1" pad="72"/>
 <contactref element="JP2" pad="1"/>
@@
 <wire x1="42.86" y1="46.77" x2="41.51" y2="48.12" width="0.3048" layer="16"/>
 </signal>
-<signal name="N$32">
+<signal name="17">
 <contactref element="U$1" pad="57"/>
 <contactref element="JP2" pad="16"/>
@@
 <wire x1="45.36" y1="46.81" x2="44.05" y2="48.12" width="0.3048" layer="16"/>
 </signal>
-<signal name="N$33">
+<signal name="64">
 <contactref element="U$1" pad="24"/>
 <contactref element="JP3" pad="1"/>
@@
 <wire x1="7.22" y1="2.59" x2="8.49" y2="1.32" width="0.4064" layer="1"/>
 </signal>
-<signal name="N$48">
+<signal name="49">
 <contactref element="U$1" pad="9"/>
 <contactref element="JP3" pad="16"/>
@@
 <wire x1="22.206" y1="18.214" x2="22.2" y2="18.22" width="0.4064" layer="1"/>
 </signal>
-<signal name="N$49">
+<signal name="40">
 <contactref element="U$1" pad="80"/>
 <contactref element="JP4" pad="1"/>
@@
 <wire x1="13.443" y1="25.577" x2="13.5" y2="25.52" width="0.3048" layer="1"/>
 </signal>
-<signal name="N$56">
+<signal name="33">
 <contactref element="U$1" pad="73"/>
 <contactref element="JP4" pad="8"/>
@@
 <wire x1="13.392" y1="26.212" x2="13.5" y2="26.32" width="0.3048" layer="1"/>
 </signal>
-<signal name="N$57">
+<signal name="48">
 <contactref element="U$1" pad="8"/>
 <contactref element="JP5" pad="1"/>
@@
 <wire x1="16.618" y1="18.202" x2="16.6" y2="18.22" width="0.4064" layer="1"/>
 </signal>
-<signal name="N$64">
+<signal name="41">
 <contactref element="U$1" pad="1"/>
 <contactref element="JP5" pad="8"/>
@@
 </board>
 </drawing>
+<compatibility>
+<note version="6.3" minversion="6.2.2" severity="warning">
+Since Version 6.2.2 text objects can contain more than one line,
+which will not be processed correctly with this version.
+</note>
+</compatibility>
 </eagle>
