File: hv507_connector.sch (EAGLE design)
At the start: 10 parts

Commit message: * DMF board first iteration
Connections:
- net N$1 renamed 16
- net N$16 renamed 1
- net N$17 renamed 32
- net N$32 renamed 17
- net N$33 renamed 64
- net N$48 renamed 49
- net N$49 renamed 40
- net N$56 renamed 33
- net N$57 renamed 48
- net N$64 renamed 41
Other:
- moved on the sheet: JP1, JP2, JP3, JP4, JP5
